File: assets/Board/UnderfloorHeatingController/relay_pair.kicad_sch (KiCad schematic)
At the start: 7 parts, among them K2 Relay_SPST_Latching_1coil, K3 Relay_SPST_Latching_1coil, U3 DRV8833PWR

Commit message: Fully routed board.
Parts:
- removed R13: 47k, Resistor_SMD:R_0805_2012Metric_Pad1.20x1.40mm_HandSolder, symbol Device:R
- C10: value 10u -> 10uF
- C8: value 0.01u -> 0.01uF
- C9: value 2.2u -> 2.2uF
Connections:
- net +5V: now also U3.1 (~{SLEEP})
- net at U3.2 (AOUT1): now also K2.A2; no longer K2.A1
- net at U3.4 (AOUT2): now also K2.A1; no longer K2.A2
Other:
- moved on the sheet: C8
Changed lines of the file:
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@@
 	(wire
 		(pts
-			(xy 21.59 57.15) (xy 21.59 46.99)
-		)
-		(stroke
-			(width 0)
-			(type default)
-		)
-	)
-	(wire
-		(pts
-			(xy 106.68 67.31) (xy 106.68 43.18)
-		)
-		(stroke
-			(width 0)
-			(type default)
-		)
-	)
-	(wire
-		(pts
-			(xy 48.26 54.61) (xy 50.8 54.61)
+			(xy 29.21 57.15) (xy 29.21 46.99)
+		)
+		(stroke
+			(width 0)
+			(type default)
+		)
+	)
+	(wire
+		(pts
+			(xy 76.2 69.85) (xy 106.68 69.85)
+		)
+		(stroke
+			(width 0)
+			(type default)
+		)
+	)
+	(wire
+		(pts
+			(xy 119.38 67.31) (xy 119.38 62.23)
 		)
 		(stroke
@@
 	(wire
 		(pts
-			(xy 76.2 67.31) (xy 106.68 67.31)
-		)
-		(stroke
-			(width 0)
-			(type default)
-		)
-	)
-	(wire
-		(pts
 			(xy 82.55 36.83) (xy 86.36 36.83)
 		)
@@
 	(wire
 		(pts
-			(xy 33.02 57.15) (xy 50.8 57.15)
+			(xy 40.64 57.15) (xy 50.8 57.15)
 		)
 		(stroke
@@
 	(wire
 		(pts
+			(xy 106.68 69.85) (xy 106.68 43.18)
+		)
+		(stroke
+			(width 0)
+			(type default)
+		)
+	)
+	(wire
+		(pts
 			(xy 106.68 74.93) (xy 106.68 99.06)
 		)
@@
 	(wire
 		(pts
-			(xy 40.64 54.61) (xy 35.56 54.61)
-		)
-		(stroke
-			(width 0)
-			(type default)
-		)
-	)
-	(wire
-		(pts
 			(xy 68.58 49.53) (xy 68.58 36.83)
 		)
@@
 	(wire
 		(pts
-			(xy 119.38 69.85) (xy 119.38 62.23)
-		)
-		(stroke
-			(width 0)
-			(type default)
-		)
-	)
-	(wire
-		(pts
 			(xy 132.08 41.91) (xy 132.08 46.99)
 		)
@@
 	(wire
 		(pts
-			(xy 25.4 57.15) (xy 21.59 57.15)
-		)
-		(stroke
-			(width 0)
-			(type default)
-		)
-	)
-	(wire
-		(pts
-			(xy 76.2 69.85) (xy 119.38 69.85)
+			(xy 33.02 57.15) (xy 29.21 57.15)
 		)
 		(stroke
@@
 	(wire
 		(pts
-			(xy 35.56 54.61) (xy 35.56 46.99)
+			(xy 44.45 54.61) (xy 44.45 46.99)
 		)
 		(stroke
@@
 	(wire
 		(pts
+			(xy 119.38 43.18) (xy 119.38 46.99)
+		)
+		(stroke
+			(width 0)
+			(type default)
+		)
+	)
+	(wire
+		(pts
 			(xy 76.2 72.39) (xy 119.38 72.39)
 		)
@@
 	(wire
 		(pts
+			(xy 44.45 54.61) (xy 50.8 54.61)
+		)
+		(stroke
+			(width 0)
+			(type default)
+		)
+	)
+	(wire
+		(pts
 			(xy 50.8 59.69) (xy 44.45 59.69)
 		)
@@
 	(wire
 		(pts
+			(xy 76.2 67.31) (xy 119.38 67.31)
+		)
+		(stroke
+			(width 0)
+			(type default)
+		)
+	)
+	(wire
+		(pts
 			(xy 71.12 36.83) (xy 71.12 49.53)
 		)
@@
 		(pts
 			(xy 38.1 69.85) (xy 50.8 69.85)
-		)
-		(stroke
-			(width 0)
-			(type default)
-		)
-	)
-	(wire
-		(pts
-			(xy 119.38 43.18) (xy 119.38 46.99)
 		)
 		(stroke
@@
 			)
 			(justify right)
-		)
-	)
-	(symbol
-		(lib_id "Device:R")
-		(at 44.45 54.61 90)
-		(unit 1)
-		(exclude_from_sim no)
-		(in_bom yes)
-		(on_board yes)
-		(dnp no)
-		(fields_autoplaced yes)
-		(property "Reference" "R13"
-			(at 44.45 48.26 90)
-			(effects
-				(font
-					(size 1.27 1.27)
-				)
-			)
-		)
-		(property "Value" "47k"
-			(at 44.45 50.8 90)
-			(effects
-				(font
-					(size 1.27 1.27)
-				)
-			)
-		)
-		(property "Footprint" "Resistor_SMD:R_0805_2012Metric_Pad1.20x1.40mm_HandSolder"
-			(at 44.45 56.388 90)
-			(effects
-				(font
-					(size 1.27 1.27)
-				)
-				(hide yes)
-			)
-		)
-		(property "Datasheet" "~"
-			(at 44.45 54.61 0)
-			(effects
-				(font
-					(size 1.27 1.27)
-				)
-				(hide yes)
-			)
-		)
-		(property "Description" "Resistor"
-			(at 44.45 54.61 0)
-			(effects
-				(font
-					(size 1.27 1.27)
-				)
-				(hide yes)
-			)
-		)
-		(pin "1"
-		)
-		(pin "2"
-		)
-		(instances
-			(project "UnderfloorHeatingController"
-				(path "/7f42c8c9-93b7-46f2-bb55-850effcdf72e/46b4c450-0b60-48c2-aa16-74b21946fd23/d29f4d68-9338-48eb-bb0d-9d66fa5e2594"
-					(reference "R14")
-					(unit 1)
-				)
-				(path "/7f42c8c9-93b7-46f2-bb55-850effcdf72e/46b4c450-0b60-48c2-aa16-74b21946fd23/ee06f143-6fc2-4883-9660-65f33d6f68e8"
-					(reference "R15")
-					(unit 1)
-				)
-				(path "/7f42c8c9-93b7-46f2-bb55-850effcdf72e/46b4c450-0b60-48c2-aa16-74b21946fd23/f32a9db5-a50f-488c-aeb7-a90f6926cec4"
-					(reference "R13")
-					(unit 1)
-				)
-			)
 		)
 	)
@@
 	(symbol
 		(lib_id "Device:C")
-		(at 29.21 57.15 90)
+		(at 36.83 57.15 90)
 		(unit 1)
 		(exclude_from_sim no)
@@
 		(fields_autoplaced yes)
 		(property "Reference" "C8"
-			(at 29.21 49.53 90)
-			(effects
-				(font
-					(size 1.27 1.27)
-				)
-			)
-		)
-		(property "Value" "0.01u"
-			(at 29.21 52.07 90)
+			(at 36.83 49.53 90)
+			(effects
+				(font
+					(size 1.27 1.27)
+				)
+			)
+		)
+		(property "Value" "0.01uF"
+			(at 36.83 52.07 90)
 			(effects
 				(font
@@
 		)
 		(property "Footprint" "Capacitor_SMD:C_0805_2012Metric_Pad1.18x1.45mm_HandSolder"
-			(at 33.02 56.1848 0)
+			(at 40.64 56.1848 0)
 			(effects
 				(font
@@
 		)
 		(property "Datasheet" "~"
-			(at 29.21 57.15 0)
+			(at 36.83 57.15 0)
 			(effects
 				(font
@@
 		)
 		(property "Description" "Unpolarized capacitor"
-			(at 29.21 57.15 0)
+			(at 36.83 57.15 0)
 			(effects
 				(font
@@
 	(symbol
 		(lib_id "power:+5V")
-		(at 35.56 46.99 0)
+		(at 44.45 46.99 0)
 		(unit 1)
 		(exclude_from_sim no)
@@
 		(fields_autoplaced yes)
 		(property "Reference" "#PWR05"
-			(at 35.56 50.8 0)
+			(at 44.45 50.8 0)
 			(effects
 				(font
@@
 		)
 		(property "Value" "+5V"
-			(at 35.56 41.91 0)
+			(at 44.45 41.91 0)
 			(effects
 				(font
@@
 		)
 		(property "Footprint" ""
-			(at 35.56 46.99 0)
+			(at 44.45 46.99 0)
 			(effects
 				(font
@@
 		)
 		(property "Datasheet" ""
-			(at 35.56 46.99 0)
+			(at 44.45 46.99 0)
 			(effects
 				(font
@@
 		)
 		(property "Description" "Power symbol creates a global label with name \"+5V\""
-			(at 35.56 46.99 0)
+			(at 44.45 46.99 0)
 			(effects
 				(font
@@
 	(symbol
 		(lib_id "power:+5V")
-		(at 21.59 46.99 0)
+		(at 29.21 46.99 0)
 		(unit 1)
 		(exclude_from_sim no)
@@
 		(fields_autoplaced yes)
 		(property "Reference" "#PWR04"
-			(at 21.59 50.8 0)
+			(at 29.21 50.8 0)
 			(effects
 				(font
@@
 		)
 		(property "Value" "+5V"
-			(at 21.59 41.91 0)
+			(at 29.21 41.91 0)
 			(effects
 				(font
@@
 		)
 		(property "Footprint" ""
-			(at 21.59 46.99 0)
+			(at 29.21 46.99 0)
 			(effects
 				(font
@@
 		)
 		(property "Datasheet" ""
-			(at 21.59 46.99 0)
+			(at 29.21 46.99 0)
 			(effects
 				(font
@@
 		)
 		(property "Description" "Power symbol creates a global label with name \"+5V\""
-			(at 21.59 46.99 0)
+			(at 29.21 46.99 0)
 			(effects
 				(font
@@
 			)
 		)
-		(property "Value" "2.2u"
+		(property "Value" "2.2uF"
 			(at 60.96 31.75 90)
 			(effects
@@
 			)
 		)
-		(property "Value" "10u"
+		(property "Value" "10uF"
 			(at 78.74 31.75 90)
 			(effects
