File: assets/Board/UnderfloorHeatingController/eta_relays.kicad_sch (KiCad schematic)
At the start: 12 parts, among them J1 Screw_Terminal_01x02, J10 Screw_Terminal_01x02, J11 Screw_Terminal_01x02, J12 Screw_Terminal_01x02, J13 Screw_Terminal_01x02, J14 Screw_Terminal_01x02, J4 Screw_Terminal_01x02, J5 Screw_Terminal_01x02, J6 Screw_Terminal_01x02, J7 Screw_Terminal_01x02, J8 Screw_Terminal_01x02, J9 Screw_Terminal_01x02

Commit message: Improved routing and layout.
Connections:
- net Relay pair - ETA1/POWER_RELAY_A: now also J4.1 (Pin_1), J6.1 (Pin_1)
- net Relay pair - ETA1/POWER_RELAY_B: now also J8.1 (Pin_1); no longer J4.1 (Pin_1), J6.1 (Pin_1)
- net Relay pair - ETA2/POWER_RELAY_A: no longer J8.1 (Pin_1)
- net Relay pair - ETA2/POWER_RELAY_B: no longer J10.1 (Pin_1)
- net Relay pair - ETA3/POWER_RELAY_A: now also J10.1 (Pin_1); no longer J11.1 (Pin_1), J13.1 (Pin_1)
- net Relay pair - ETA3/POWER_RELAY_B: now also J11.1 (Pin_1), J13.1 (Pin_1)
Other:
- moved on the sheet: J10, J11, J12, J13, J14, J5, J6, J7, J8, J9
